File: electronica/puente_h/puente_h.brd (EAGLE design)
At the start: 78.7 x 127.6 mm, 40 parts, among them IC1 7805, IC2 7812, IC3 7404LP, IC4 7408LP, IC5 ADUM1400, Q1 IRF2804, Q2 IRF2804, Q5 IRF2804, Q6 IRF2804, U1 IR2110LP

Commit message: puente h ok
Routing:
- net VIN: track 77.3 -> 122.6 mm
- net N$12: track 38.9 -> 40.5 mm
- net SD: track 32.3 -> 33.8 mm
- net N$35: track 89.3 -> 87.9 mm
- net N$11: track 24.2 -> 25.1 mm
- net +12V: track 151.8 -> 150.9 mm
Other:
- board size 78.7 x 127.6 mm -> 78.7 x 132.2 mm
